File: HagiwoKick.kicad_sch (KiCad schematic)
At the start: 37 parts, among them J1 Tune CV, J2 Eurorack_Power_16pin_Shrouded, J3 Out, J4 Trig

Commit message: latest updates
Parts:
- removed J1: Tune CV, Library:EighthInch_PJ398SM_T_TN_S, symbol Connector_Audio:AudioJack2_SwitchT
- removed J2: Eurorack_Power_16pin_Shrouded, PCM_4ms_Connector:Pins_2x08_2.54mm_TH_EuroPower_Shrouded, symbol PCM_4ms_Connector:Eurorack_Power_16pin_Shrouded
- removed J3: Out, Library:EighthInch_PJ398SM_T_TN_S, symbol Connector_Audio:AudioJack2_SwitchT
- removed J4: Trig, Library:EighthInch_PJ398SM_T_TN_S, symbol Connector_Audio:AudioJack2_SwitchT
- added J1: TUNE CV, Library:EighthInch_PJ398SM_3mmNPTH, symbol PCM_4ms_Jack:3.5mm_Mono_Switched_sm
- added J2: OUT, Library:EighthInch_PJ398SM_3mmNPTH, symbol PCM_4ms_Jack:3.5mm_Mono_Switched_sm
- added J3: TRIG, Library:EighthInch_PJ398SM_3mmNPTH, symbol PCM_4ms_Jack:3.5mm_Mono_Switched_sm
- added PWR1: Eurorack_Power_10pin_Unshrouded, Library:IDC-Header_2x05_P2.54mm_Vertical_Euro_Power_Striped_ThickerText, symbol PCM_4ms_Connector:Eurorack_Power_10pin_Unshrouded
- C1, C2, C3, C4, C5: value 100pF (101) -> 100pF; Silkscreen Value (none) -> 101▼
- C10: value 2.2nF (222) -> 2.2nF; Silkscreen Value (none) -> 222▼
- C6: value 100nF (104) -> 100nF; Silkscreen Value (none) -> 104▼
- C7: footprint Capacitor_THT:CP_Radial_D6.3mm_P2.50mm -> Capacitor_THT:CP_Radial_D4.0mm_P1.50mm; Silkscreen Value (none) -> 10uF▼
- C8: value 2.2uF (225) -> 2.2uF; Silkscreen Value (none) -> 225▼
- C9: value 470nF (474) -> 470nF; Silkscreen Value (none) -> 474▼
- D1, D2, D3, D4, D5, D6: footprint Diode_THT:D_DO-35_SOD27_P7.62mm_Horizontal -> Library:D_DO-35_SOD27_P7.62mm_Horizontal_Widened_No_K
- D7: value LED_Filled -> LED
- R1, R10, R2, R3, R4, R5: value 1K -> 1k
- R6, R8: value 100K -> 100k
- R7: value 33K -> 33k
- RV1: renamed from Tone1; value 100K -> 100k; Silkscreen Value (none) -> TONE
- RV2: renamed from Harmonic1; value 100K -> 100k; Silkscreen Value (none) -> HARMONIC
- RV3: renamed from Attack1; value 100K -> 100k; Silkscreen Value (none) -> ATTACK
- RV4: renamed from Decay1; value 100K -> 100k; Silkscreen Value (none) -> DECAY
Connections:
- net +12V: now also PWR1.1 (+12V), PWR1.2 (+12V)
- net GND: now also J1.3 (SW), J2.3 (SW), J3.3 (SW), PWR1.3 (GND), PWR1.4 (GND), PWR1.5 (GND), PWR1.6 (GND), PWR1.7 (GND), PWR1.8 (GND)
- net at C10.2: now also J2.1 (SIG)
- net at R10.2: now also J3.1 (SIG)
- net at R5.1: now also J1.1 (SIG)
- new net -12V: PWR1.10 (-12V), PWR1.9 (-12V)
Other:
- moved on the sheet: C6, C7

Commit message: v1.1 ready for final check
Parts:
- C7: footprint Capacitor_THT:CP_Radial_D4.0mm_P1.50mm -> Capacitor_THT:CP_Radial_D4.0mm_P2.00mm
- RV1, RV2, RV3, RV4: value 100k -> 100k B
Changed lines of the file:
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@@
 			)
 		)
-		(property "Value" "100k"
+		(property "Value" "100k B"
 			(at 29.21 58.4199 0)
 			(effects
@@
 			)
 		)
-		(property "Footprint" "Capacitor_THT:CP_Radial_D4.0mm_P1.50mm"
+		(property "Footprint" "Capacitor_THT:CP_Radial_D4.0mm_P2.00mm"
 			(at 162.2552 132.08 0)
 			(effects
@@
 			)
 		)
-		(property "Value" "100k"
+		(property "Value" "100k B"
 			(at 29.21 80.0099 0)
 			(effects
@@
 			)
 		)
-		(property "Value" "100k"
+		(property "Value" "100k B"
 			(at 29.21 36.8299 0)
 			(effects
@@
 			)
 		)
-		(property "Value" "100k"
+		(property "Value" "100k B"
 			(at 29.21 101.5999 0)
 			(effects

Commit message: updating after Dmitri's changes
Parts:
- R11, R9: Silkscreen Value (none) -> 470Ω
Changed lines of the file:
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@@
+			)
+		)
+		(property "Silkscreen Value" "470Ω"
+			(at 181.61 39.37 90)
+			(effects
+				(font
+					(size 1.27 1.27)
+				)
+				(hide yes)
 			)
 		)
@@
 			(effects
 				(font
+					(size 1.27 1.27)
+				)
+				(hide yes)
+			)
+		)
+		(property "Silkscreen Value" "470Ω"
+			(at 199.39 39.37 90)
+			(effects
+				(font

Commit message: switched positions of TRIG and OUT outputs
Parts:
- J1: value TUNE CV -> TUNECV
Changed lines of the file:
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@@
 			)
 		)
-		(property "Value" "TUNE CV"
+		(property "Value" "TUNECV"
 			(at 29.21 125.73 0)
 			(effects

Commit message: reversed orientated of pots on schematic to make +5V rightmost pin and updated routing. This completes v1.2
Connections:
- net +5V: now also RV1.3, RV2.3, RV3.3, RV4.3; no longer RV1.1, RV2.1, RV3.1, RV4.1
- net GND: now also RV1.1, RV2.1, RV3.1, RV4.1; no longer RV1.3, RV2.3, RV3.3, RV4.3
Changed lines of the file:
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@@
 		(lib_id "Device:R_Potentiometer")
 		(at 31.75 57.15 0)
+		(mirror x)
 		(unit 1)
 		(exclude_from_sim no)
@@
 		(dnp no)
 		(property "Reference" "RV2"
-			(at 29.21 55.8799 0)
+			(at 29.21 58.4201 0)
 			(effects
 				(font
@@
 		)
 		(property "Value" "100k B"
-			(at 29.21 58.4199 0)
+			(at 29.21 55.8801 0)
 			(effects
 				(font
@@
 		)
 		(property "Silkscreen Value" "HARMONIC"
-			(at 24.384 60.96 0)
+			(at 24.384 53.34 0)
 			(effects
 				(font
@@
 		(lib_id "Device:R_Potentiometer")
 		(at 31.75 78.74 0)
+		(mirror x)
 		(unit 1)
 		(exclude_from_sim no)
@@
 		(dnp no)
 		(property "Reference" "RV3"
-			(at 29.21 77.4699 0)
+			(at 29.21 80.0101 0)
 			(effects
 				(font
@@
 		)
 		(property "Value" "100k B"
-			(at 29.21 80.0099 0)
+			(at 29.21 77.4701 0)
 			(effects
 				(font
@@
 		)
 		(property "Silkscreen Value" "ATTACK"
-			(at 25.908 82.804 0)
+			(at 25.908 74.676 0)
 			(effects
 				(font
@@
 		(lib_id "Device:R_Potentiometer")
 		(at 31.75 35.56 0)
+		(mirror x)
 		(unit 1)
 		(exclude_from_sim no)
@@
 		(dnp no)
 		(property "Reference" "RV1"
-			(at 29.21 34.2899 0)
+			(at 29.21 36.8301 0)
 			(effects
 				(font
@@
 		)
 		(property "Value" "100k B"
-			(at 29.21 36.8299 0)
+			(at 29.21 34.2901 0)
 			(effects
 				(font
@@
 		)
 		(property "Silkscreen Value" "TONE"
-			(at 26.67 39.37 0)
+			(at 26.67 31.75 0)
 			(effects
 				(font
@@
 		(lib_id "Device:R_Potentiometer")
 		(at 31.75 100.33 0)
+		(mirror x)
 		(unit 1)
 		(exclude_from_sim no)
@@
 		(dnp no)
 		(property "Reference" "RV4"
-			(at 29.21 99.0599 0)
+			(at 29.21 101.6001 0)
 			(effects
 				(font
@@
 		)
 		(property "Value" "100k B"
-			(at 29.21 101.5999 0)
+			(at 29.21 99.0601 0)
 			(effects
 				(font
@@
 		)
 		(property "Silkscreen Value" "DECAY"
-			(at 26.162 104.394 0)
-			(effects
-				(font
+			(at 26.162 96.266 0)
+			(effects
+				(font

Commit message: corrected silkscreening issue that TUNE should be TONE and other minor fixed for v1.3
Parts:
- J1: value TUNECV -> HARMCV
Connections:
- net GND: now also J1.2 (SHEILD), J2.2 (SHEILD), J3.2 (SHEILD); no longer J1.3 (SW), J2.3 (SW), J3.3 (SW)
Other:
- note added: "Sounds way louder/beefier without C10 filter cap, but with high frequency aliasing noise!"
Changed lines of the file:
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@@
 	)
 	(no_connect
-		(at 234.95 49.53)
-	)
-	(no_connect
 		(at 143.51 59.69)
 	)
@@
 	)
 	(no_connect
+		(at 228.6 43.18)
+	)
+	(no_connect
 		(at 118.11 62.23)
 	)
@@
 	)
 	(no_connect
-		(at 118.11 49.53)
+		(at 228.6 72.39)
 	)
 	(no_connect
-		(at 25.4 138.43)
+		(at 118.11 49.53)
 	)
 	(no_connect
-		(at 118.11 69.85)
+		(at 31.75 132.08)
 	)
 	(no_connect
-		(at 234.95 78.74)
+		(at 118.11 69.85)
 	)
 	(no_connect
@@
 	(wire
 		(pts
+			(xy 228.6 46.99) (xy 228.6 49.53)
+		)
+		(stroke
+			(width 0)
+			(type default)
+		)
+	)
+	(wire
+		(pts
 			(xy 35.56 78.74) (xy 41.91 78.74)
 		)
@@
 	(wire
 		(pts
-			(xy 31.75 132.08) (xy 43.18 132.08)
-		)
-		(stroke
-			(width 0)
-			(type default)
-		)
-	)
-	(wire
-		(pts
 			(xy 138.43 129.54) (xy 138.43 132.08)
 		)
@@
 	(wire
 		(pts
-			(xy 228.6 43.18) (xy 228.6 46.99)
-		)
-		(stroke
-			(width 0)
-			(type default)
-		)
-	)
-	(wire
-		(pts
 			(xy 125.73 124.46) (xy 138.43 124.46)
 		)
@@
 	(wire
 		(pts
-			(xy 226.06 72.39) (xy 228.6 72.39)
+			(xy 39.37 64.77) (xy 39.37 60.96)
 		)
 		(stroke
@@
 	(wire
 		(pts
-			(xy 39.37 64.77) (xy 39.37 60.96)
+			(xy 161.29 68.58) (xy 167.64 68.58)
 		)
 		(stroke
@@
 	(wire
 		(pts
-			(xy 161.29 68.58) (xy 167.64 68.58)
+			(xy 125.73 134.62) (xy 138.43 134.62)
 		)
 		(stroke
@@
 	(wire
 		(pts
-			(xy 125.73 134.62) (xy 138.43 134.62)
+			(xy 228.6 49.53) (xy 234.95 49.53)
 		)
 		(stroke
@@
 		)
 	)
+	(text "Sounds way louder/beefier without C10 filter cap,\nbut with high frequency aliasing noise!"
+		(exclude_from_sim no)
+		(at 219.202 26.924 0)
+		(effects
+			(font
+				(size 1.27 1.27)
+			)
+		)
+	)
 	(global_label "D3"
 		(shape input)
@@
 			)
 		)
-		(property "Value" "TUNECV"
+		(property "Value" "HARMCV"
 			(at 29.21 125.73 0)
 			(effects
@@
 	)
 	(symbol
+		(lib_id "power:GND")
+		(at 25.4 138.43 0)
+		(unit 1)
+		(exclude_from_sim no)
+		(in_bom yes)
+		(on_board yes)
+		(dnp no)
+		(fields_autoplaced yes)
+		(property "Reference" "#PWR09"
+			(at 25.4 144.78 0)
+			(effects
+				(font
+					(size 1.27 1.27)
+				)
+				(hide yes)
+			)
+		)
+		(property "Value" "GND"
+			(at 25.4 143.51 0)
+			(effects
+				(font
+					(size 1.27 1.27)
+				)
+			)
+		)
+		(property "Footprint" ""
+			(at 25.4 138.43 0)
+			(effects
+				(font
+					(size 1.27 1.27)
+				)
+				(hide yes)
+			)
+		)
+		(property "Datasheet" ""
+			(at 25.4 138.43 0)
+			(effects
+				(font
+					(size 1.27 1.27)
+				)
+				(hide yes)
+			)
+		)
+		(property "Description" "Power symbol creates a global label with name \"GND\" , ground"
+			(at 25.4 138.43 0)
+			(effects
+				(font
+					(size 1.27 1.27)
+				)
+				(hide yes)
+			)
+		)
+		(pin "1"
+		)
+		(instances
+			(project "HagiwoKick"
+				(path "/599a98da-a4a2-4635-97eb-f901b14811e2"
+					(reference "#PWR09")
+					(unit 1)
+				)
+			)
+		)
+	)
+	(symbol
 		(lib_id "power:+12V")
 		(at 138.43 134.62 180)
@@
 	(symbol
 		(lib_id "power:GND")
-		(at 43.18 132.08 0)
-		(unit 1)
-		(exclude_from_sim no)
-		(in_bom yes)
-		(on_board yes)
-		(dnp no)
-		(fields_autoplaced yes)
-		(property "Reference" "#PWR09"
-			(at 43.18 138.43 0)
-			(effects
-				(font
-					(size 1.27 1.27)
-				)
-				(hide yes)
-			)
-		)
-		(property "Value" "GND"
-			(at 43.18 137.16 0)
-			(effects
-				(font
-					(size 1.27 1.27)
-				)
-			)
-		)
-		(property "Footprint" ""
-			(at 43.18 132.08 0)
-			(effects
-				(font
-					(size 1.27 1.27)
-				)
-				(hide yes)
-			)
-		)
-		(property "Datasheet" ""
-			(at 43.18 132.08 0)
-			(effects
-				(font
-					(size 1.27 1.27)
-				)
-				(hide yes)
-			)
-		)
-		(property "Description" "Power symbol creates a global label with name \"GND\" , ground"
-			(at 43.18 132.08 0)
-			(effects
-				(font
-					(size 1.27 1.27)
-				)
-				(hide yes)
-			)
-		)
-		(pin "1"
-		)
-		(instances
-			(project "HagiwoKick"
-				(path "/599a98da-a4a2-4635-97eb-f901b14811e2"
-					(reference "#PWR09")
-					(unit 1)
-				)
-			)
-		)
-	)
-	(symbol
-		(lib_id "power:GND")
 		(at 130.81 80.01 0)
 		(unit 1)
@@
 	)
 	(symbol
-		(lib_id "power:GND")
-		(at 226.06 72.39 0)
-		(unit 1)
-		(exclude_from_sim no)
-		(in_bom yes)
-		(on_board yes)
-		(dnp no)
-		(fields_autoplaced yes)
-		(property "Reference" "#PWR024"
-			(at 226.06 78.74 0)
-			(effects
-				(font
-					(size 1.27 1.27)
-				)
-				(hide yes)
-			)
-		)
-		(property "Value" "GND"
-			(at 226.06 77.47 0)
-			(effects
-				(font
-					(size 1.27 1.27)
-				)
-			)
-		)
-		(property "Footprint" ""
-			(at 226.06 72.39 0)
-			(effects
-				(font
-					(size 1.27 1.27)
-				)
-				(hide yes)
-			)
-		)
-		(property "Datasheet" ""
-			(at 226.06 72.39 0)
-			(effects
-				(font
-					(size 1.27 1.27)
-				)
-				(hide yes)
-			)
-		)
-		(property "Description" "Power symbol creates a global label with name \"GND\" , ground"
-			(at 226.06 72.39 0)
-			(effects
-				(font
-					(size 1.27 1.27)
-				)
-				(hide yes)
-			)
-		)
-		(pin "1"
-		)
-		(instances
-			(project "HagiwoKick"
-				(path "/599a98da-a4a2-4635-97eb-f901b14811e2"
-					(reference "#PWR024")
-					(unit 1)
-				)
-			)
-		)
-	)
-	(symbol
 		(lib_id "Device:C")
 		(at 55.88 60.96 0)
@@
 					(unit 1)
 				)
+			)
+		)
+	)
+	(symbol
+		(lib_id "power:GND")
+		(at 234.95 78.74 0)
+		(unit 1)
+		(exclude_from_sim no)
+		(in_bom yes)
+		(on_board yes)
+		(dnp no)
+		(fields_autoplaced yes)
+		(property "Reference" "#PWR024"
+			(at 234.95 85.09 0)
+			(effects
+				(font
+					(size 1.27 1.27)
+				)
+				(hide yes)
+			)
+		)
+		(property "Value" "GND"
+			(at 234.95 83.82 0)
+			(effects
+				(font
+					(size 1.27 1.27)
+				)
+			)
+		)
+		(property "Footprint" ""
+			(at 234.95 78.74 0)
+			(effects
+				(font
+					(size 1.27 1.27)
+				)
+				(hide yes)
+			)
+		)
+		(property "Datasheet" ""
+			(at 234.95 78.74 0)
+			(effects
+				(font
+					(size 1.27 1.27)
+				)
+				(hide yes)
+			)
+		)
+		(property "Description" "Power symbol creates a global label with name \"GND\" , ground"
+			(at 234.95 78.74 0)
+			(effects
+				(font
+					(size 1.27 1.27)
+				)
+				(hide yes)
+			)
+		)
+		(pin "1"
+		)
+		(instances
+			(project "HagiwoKick"
+				(path "/599a98da-a4a2-4635-97eb-f901b14811e2"
+					(reference "#PWR024")
+					(unit 1)
+				)
